File: SBC.brd (EAGLE design)
At the start: 140.3 x 67.3 mm, 42 parts, among them IC1 MAX3232CPE, IC2 74LS04N, IC3 74LS00N, IC5 NE555P, J1 POWER_JACKPTH, J2 COMPUTER-PERIPHERAL-POWERRA, J3 22-27-2021-02

Commit message: Added gerber files
Parts:
- C7: value (none) -> 10uF
- RAM: value (none) -> 62256
- moved X1 80.2 mm to (187.0, 31.1)
- moved C1 79.9 mm to (212.1, 40.6)
- moved C2 79.9 mm to (212.1, 47.0)
- moved C3 79.9 mm to (162.6, 31.0)
- moved C4 79.9 mm to (162.6, 33.6)
- moved C5 79.9 mm to (214.0, 56.9)
- moved IC2 79.9 mm to (160.0, 44.5)
- moved IC4 79.9 mm to (219.7, 36.8)
- moved VIA0A 79.9 mm to (128.3, 25.4)
- moved VIA0B 79.9 mm to (128.3, 31.8)
- moved C6 79.9 mm to (144.8, 33.0)
- moved J3 79.9 mm to (150.2, 33.3)
- moved Q1 79.9 mm to (156.2, 33.9)
- moved R1 79.9 mm to (156.2, 27.9)
- moved R2 79.9 mm to (166.4, 25.4)
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Connections:
- removed net N$32: IC1.11
- removed net N$33: ACIA.5, IC1.14
- removed net RINGINDICATOR: X1.9
- removed net TRANSMITDATA: IC1.9, X1.3
- removed net VSS: RAM.14
- new net DATASETREADY: ACIA.17, X1.6
- new net N$1: LED1.K, R5.P$1
- new net N$3: IC1.14, X1.3
- new net N$5: ACIA.28, CPU.34
- new net N$7: ACIA.10, IC1.11
- new net N$8: ACIA.12, IC1.12
- net DATACARRIERDETECT: now also ACIA.16; no longer X1.6
- net DTEREADY: no longer IC1.8
- net GND: now also RAM.14, X1.9; no longer ACIA.16, ACIA.17
- net IRQ: now also ACIA.26, VIA0.21
- net N$17: now also VIA0.23
- net RECEIVEDATA: now also IC1.13
- net VCC: no longer LED1.K, R5.P$1
Routing:
- net IRQ: track 2.54 -> 216.9 mm, vias 0 -> 7
- net GND: track 107.6 -> 284.4 mm, vias 2 -> 8
- net N$17: track 0.00 -> 143.8 mm, vias 0 -> 4
- net PHI2: track 84.9 -> 190.4 mm, vias 2 -> 6
- net N$6: track 36.4 -> 138.9 mm, vias 0 -> 4
- net ADDRESS15: track 100.7 -> 199.9 mm, vias 2 -> 6
- net N$1: track 0.00 -> 84.0 mm, vias 0 -> 1
- net DATASETREADY: track 0.00 -> 76.0 mm, vias 0 -> 3
- net VCC: track 79.1 -> 153.5 mm, vias 2 -> 5
- net N$5: track 0.00 -> 67.7 mm, vias 0 -> 3
- net DATACARRIERDETECT: track 3.42 -> 64.0 mm, vias 0 -> 4
- net N$26: track 0.00 -> 57.5 mm, vias 0 -> 2
- net N$8: track 0.00 -> 40.9 mm, vias 0 -> 2
- net TRANSMITDATA: track 39.6 -> 0.00 mm, vias 1 -> 0
- net ADDRESS10: track 49.6 -> 87.0 mm
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- added copper zone on layer 16, net GND
- added copper zone on layer 1, net VCC

Commit message: Fixed issue with SMD switch
Updated schematic, board, BOM & gerbers for through-hole switch. Sent
gerber off to production.
Parts:
- S2: device SparkFun-Electromechanical:SWITCH-SPDT-SMD -> SparkFun-Electromechanical:SWITCH-SPDT_LOCK.007S
- moved S2 6.02 mm to (219.1, 48.9), turned to 0 degrees
- moved LED1 5.90 mm to (224.1, 49.2), turned to 0 degrees
- moved R6 1.91 mm to (220.3, 59.7)
- moved Q2 1.27 mm to (224.2, 59.1)
Connections:
- removed net N$28: IC4.OUT, LED1.A, S2.3
- new net N$32: IC4.OUT, S2.3
- net VCC: now also LED1.A
Routing:
- net VCC: track 153.5 -> 137.3 mm
- net N$28: track 13.0 -> 0.00 mm
- net N$1: track 84.0 -> 77.2 mm
- net N$32: track 0.00 -> 6.33 mm
- net N$30: track 15.2 -> 17.1 mm
- net N$31: track 22.4 -> 20.8 mm
- net GND: track 284.4 -> 283.1 mm
Other:
- board text added: "Benchoff Mar 2013"
- board text added: "OFF"
- board text added: "ON"
Changed lines of the file:
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@@
 <setting verticaltext="up"/>
 </settings>
-<grid distance="0.05" unitdist="inch" unit="inch" style="lines" multiple="1" display="no" altdistance="0.025" altunitdist="inch" altunit="inch"/>
+<grid distance="0.05" unitdist="inch" unit="inch" style="lines" multiple="1" display="no" altdistance="0.012" altunitdist="inch" altunit="inch"/>
 <layers>
 <layer number="1" name="Top" color="4" fill="1" visible="yes" active="yes"/>
@@
 <rectangle x1="219.1386" y1="79.24145" x2="221.21378125" y2="79.2836125" layer="1"/>
 <rectangle x1="219.6466" y1="79.2836125" x2="220.9166" y2="79.32603125" layer="1"/>
+<text x="221.615" y="45.085" size="1.778" layer="21" font="vector" ratio="18">ON</text>
+<text x="221.5896" y="51.5112" size="1.778" layer="21" font="vector" ratio="18">OFF</text>
+<text x="175.006" y="22.86" size="1.778" layer="21" font="vector" ratio="18">Benchoff Mar 2013</text>
 </plain>
 <attributes>
@@
 <element name="R4" library="SparkFun-Resistors" package="AXIAL-0.3" value="47k" x="165.1" y="34.29" rot="R270"/>
 <element name="D1" library="SparkFun-DiscreteSemi" package="DIODE-1N4148" value="" x="156.21" y="25.4254"/>
-<element name="S2" library="SparkFun-Electromechanical" package="SWITCH-SPDT-SMD" value="" x="224.79" y="46.99" rot="R270"/>
-<element name="LED1" library="led" package="LED3MM" value="" x="218.44" y="50.7746" rot="R90"/>
+<element name="LED1" library="led" package="LED3MM" value="" x="224.1296" y="49.1998"/>
 <element name="R5" library="SparkFun-Passives" package="AXIAL-0.3EZ" value="150" x="167.64" y="34.29" rot="R90"/>
 <element name="C8" library="SparkFun-Capacitors" package="CAP-PTH-SMALLEZ" value="47pf" x="217.17" y="62.865" rot="R180"/>
 <element name="C9" library="SparkFun-Capacitors" package="CAP-PTH-SMALLEZ" value="47pf" x="217.17" y="59.69" rot="R180"/>
-<element name="Q2" library="crystal" package="HC49/S" value="" x="224.155" y="57.785" rot="R90">
-<attribute name="OC_NEWARK" value="unknown" x="328.295" y="141.605" size="1.778" layer="27" rot="R90" display="off"/>
-<attribute name="MPN" value="" x="328.295" y="141.605" size="1.778" layer="27" rot="R90" display="off"/>
-<attribute name="MF" value="" x="328.295" y="141.605" size="1.778" layer="27" rot="R90" display="off"/>
-<attribute name="OC_FARNELL" value="1667008" x="328.295" y="141.605" size="1.778" layer="27" rot="R90" display="off"/>
+<element name="Q2" library="crystal" package="HC49/S" value="" x="224.155" y="59.055" rot="R90">
+<attribute name="OC_NEWARK" value="unknown" x="328.295" y="142.875" size="1.778" layer="27" rot="R90" display="off"/>
+<attribute name="MPN" value="" x="328.295" y="142.875" size="1.778" layer="27" rot="R90" display="off"/>
+<attribute name="MF" value="" x="328.295" y="142.875" size="1.778" layer="27" rot="R90" display="off"/>
+<attribute name="OC_FARNELL" value="1667008" x="328.295" y="142.875" size="1.778" layer="27" rot="R90" display="off"/>
 </element>
-<element name="R6" library="SparkFun-Passives" package="AXIAL-0.3EZ" value="180k" x="220.345" y="57.785" rot="R270"/>
+<element name="R6" library="SparkFun-Passives" package="AXIAL-0.3EZ" value="180k" x="220.345" y="59.69" rot="R270"/>
 <element name="R7" library="SparkFun-Resistors" package="AXIAL-0.3EZ" value="3.3k" x="170.18" y="34.29" rot="R270"/>
 <element name="R8" library="SparkFun-Resistors" package="AXIAL-0.3EZ" value="3.3k" x="166.37" y="27.94"/>
@@
 <attribute name="OC_FARNELL" value="unknown" x="150.1902" y="33.3248" size="1.778" layer="27" rot="R90" display="off"/>
 </element>
+<element name="S2" library="SparkFun-Electromechanical" package="SWITCH-SPDT_LOCK.007S" value="" x="219.075" y="48.895"/>
 </elements>
 <signals>
@@
 <wire x1="217.71" y1="29.75" x2="219.71" y2="31.75" width="2.1844" layer="1"/>
 <wire x1="219.71" y1="31.75" x2="219.71" y2="40.64" width="2.1844" layer="1"/>
-<wire x1="219.71" y1="41.91" x2="219.71" y2="40.64" width="2.1844" layer="1"/>
 <wire x1="106.68" y1="35.56" x2="106.68" y2="36.83" width="0.3048" layer="16"/>
 <wire x1="106.68" y1="36.83" x2="105.41" y2="38.1" width="0.3048" layer="16"/>
@@
 <contactref element="R4" pad="P$2"/>
 <contactref element="D1" pad="C"/>
-<contactref element="S2" pad="2"/>
 <contactref element="CPU" pad="2"/>
 <contactref element="R7" pad="P$2"/>
@@
 <wire x1="190.5" y1="47.2948" x2="190.5" y2="48.26" width="0.3048" layer="16"/>
 <via x="110.49" y="35.56" extent="1-16" drill="1.3" alwaysstop="yes"/>
-<contactref element="J2" pad="5V"/>
-<wire x1="222.04" y1="46.99" x2="220.98" y2="46.99" width="0.3048" layer="1"/>
-<wire x1="220.98" y1="46.99" x2="219.71" y2="48.26" width="0.3048" layer="1"/>
-<wire x1="219.71" y1="48.26" x2="219.71" y2="50.7746" width="0.3048" layer="1"/>
 <wire x1="160.02" y1="25.4254" x2="160.3502" y2="25.7302" width="0.3048" layer="1"/>
 <wire x1="160.3502" y1="25.7302" x2="161.29" y2="26.67" width="0.3048" layer="1"/>
@@
 <wire x1="163.83" y1="26.67" x2="165.1" y2="27.94" width="0.3048" layer="1"/>
 <contactref element="RAM" pad="28"/>
-<wire x1="218.4146" y1="52.0446" x2="215.9" y2="49.53" width="0.3048" layer="16"/>
-<wire x1="215.9" y1="49.53" x2="215.9" y2="45.0088" width="0.3048" layer="16"/>
-<wire x1="215.9" y1="45.0088" x2="215.1888" y2="44.2976" width="0.3048" layer="16"/>
-<wire x1="219.71" y1="50.7746" x2="219.6846" y2="50.7746" width="0.4064" layer="1"/>
-<wire x1="219.6846" y1="50.7746" x2="218.4146" y2="52.0446" width="0.4064" layer="1"/>
 <polygon width="0.4064" layer="1">
 <vertex x="224.79" y="88.9"/>
@@
 <wire x1="166.37" y1="27.94" x2="170.18" y2="27.94" width="0.4064" layer="16"/>
 <wire x1="168.91" y1="82.55" x2="168.91" y2="85.09" width="0.4064" layer="16"/>
+<contactref element="S2" pad="2"/>
+<contactref element="J2" pad="5V"/>
+<contactref element="LED1" pad="A"/>
 </signal>
 <signal name="ADDRESS0">
@@
 <wire x1="167.64" y1="47.5996" x2="167.64" y2="48.26" width="0.3048" layer="1"/>
 </signal>
-<signal name="N$28">
-<contactref element="S2" pad="3"/>
-<contactref element="IC4" pad="OUT"/>
-<contactref element="LED1" pad="A"/>
-<wire x1="218.44" y1="44.45" x2="222" y2="44.45" width="0.3048" layer="1"/>
-<wire x1="222" y1="44.45" x2="222.04" y2="44.49" width="0.3048" layer="1"/>
-<wire x1="218.44" y1="49.5046" x2="218.44" y2="44.45" width="0.3048" layer="1"/>
-<wire x1="217.17" y1="40.64" x2="217.17" y2="43.18" width="0.4064" layer="1"/>
-<wire x1="217.17" y1="43.18" x2="218.44" y2="44.45" width="0.4064" layer="1"/>
-</signal>
 <signal name="N$30">
 <contactref element="C8" pad="2"/>
@@
 <contactref element="R6" pad="P$1"/>
 <contactref element="ACIA" pad="6"/>
-<wire x1="220.345" y1="61.595" x2="222.758" y2="61.595" width="0.3048" layer="1"/>
-<wire x1="222.758" y1="61.595" x2="224.155" y2="60.198" width="0.3048" layer="1"/>
-<wire x1="220.345" y1="61.595" x2="215.9" y2="61.595" width="0.3048" layer="16"/>
+<wire x1="220.345" y1="63.5" x2="224.028" y2="61.595" width="0.3048" layer="1"/>
+<wire x1="224.028" y1="61.595" x2="224.155" y2="61.468" width="0.3048" layer="1"/>
 <wire x1="215.9" y1="61.595" x2="214.63" y2="62.865" width="0.3048" layer="16"/>
 <wire x1="214.63" y1="62.865" x2="212.725" y2="62.865" width="0.3048" layer="16"/>
 <wire x1="212.725" y1="62.865" x2="210.82" y2="64.77" width="0.3048" layer="16"/>
+<wire x1="215.9" y1="61.595" x2="220.345" y2="61.595" width="0.3048" layer="16"/>
+<wire x1="220.345" y1="61.595" x2="220.345" y2="63.5" width="0.3048" layer="16"/>
 </signal>
 <signal name="N$31">
@@
 <contactref element="R6" pad="P$2"/>
 <contactref element="ACIA" pad="7"/>
-<wire x1="220.345" y1="53.975" x2="222.758" y2="53.975" width="0.3048" layer="1"/>
-<wire x1="222.758" y1="53.975" x2="224.155" y2="55.372" width="0.3048" layer="1"/>
+<wire x1="220.345" y1="55.88" x2="222.758" y2="55.88" width="0.3048" layer="1"/>
+<wire x1="222.758" y1="55.88" x2="224.155" y2="56.642" width="0.3048" layer="1"/>
 <wire x1="210.82" y1="67.31" x2="212.09" y2="67.31" width="0.3048" layer="1"/>
 <wire x1="212.09" y1="67.31" x2="213.36" y2="66.04" width="0.3048" layer="1"/>
 <wire x1="213.36" y1="66.04" x2="213.36" y2="60.96" width="0.3048" layer="1"/>
 <wire x1="213.36" y1="60.96" x2="214.63" y2="59.69" width="0.3048" layer="1"/>
-<wire x1="214.63" y1="59.69" x2="220.345" y2="53.975" width="0.3048" layer="1"/>
+<wire x1="214.63" y1="59.69" x2="220.345" y2="55.88" width="0.3048" layer="1"/>
 </signal>
 <signal name="PHI2">
@@
 <contactref element="R5" pad="P$1"/>
 <contactref element="LED1" pad="K"/>
-<wire x1="218.44" y1="52.0446" x2="222.9358" y2="52.0446" width="0.4064" layer="16"/>
-<wire x1="222.9358" y1="52.0446" x2="224.028" y2="50.9524" width="0.4064" layer="16"/>
-<wire x1="224.028" y1="50.9524" x2="224.028" y2="33.8836" width="0.4064" layer="16"/>
+<wire x1="225.3996" y1="49.1998" x2="224.2058" y2="48.8696" width="0.4064" layer="16"/>
+<wire x1="224.2058" y1="48.8696" x2="224.028" y2="48.4124" width="0.4064" layer="16"/>
+<wire x1="224.028" y1="48.4124" x2="224.028" y2="33.8836" width="0.4064" layer="16"/>
 <wire x1="224.028" y1="33.8836" x2="223.1136" y2="32.9692" width="0.4064" layer="16"/>
 <wire x1="223.1136" y1="32.9692" x2="211.2264" y2="32.9692" width="0.4064" layer="16"/>
@@
 <via x="219.7608" y="25.654" extent="1-16" drill="3.2"/>
 </signal>
+<signal name="N$32">
+<contactref element="IC4" pad="OUT"/>
+<contactref element="S2" pad="3"/>
+<wire x1="217.17" y1="40.64" x2="217.17" y2="44.2722" width="0.8128" layer="1"/>
+<wire x1="217.17" y1="44.2722" x2="219.075" y2="46.1772" width="0.8128" layer="1"/>
+</signal>
 </signals>
